File: hardware/panel/output-stage.kicad_pcb (KiCad board)
At the start: 2 copper layers, 20 x 128.5 mm, 11 parts

Commit message: Change extensions for kicad 6
Parts:
- removed the ? at (5.70, -61.2)
- removed the ? at (5.70, 61.2)
- removed the G*** at (0.00, 0.00) (x7)
- added ?: , Wire_Pads:SolderWirePad_single_0-8mmDrill, F.Cu at (5.70, 61.2)
- added ?: , Wire_Pads:SolderWirePad_single_0-8mmDrill, F.Cu at (5.70, -61.2)
- added G*** (x7): LOGO, LOGO, F.Cu at (0.00, 0.00)
Other:
- net class Default removed
