File: hardware/kicad-individual-channel/Stackable Mixer.kicad_pcb (KiCad board)
At the start: 2 copper layers, 20 x 110 mm, 12 parts, among them J1 L/Mono, J2 R, P1 Potentiometer_9mm_Vertical_Li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

Commit message: Changes
Parts:
- added SW1: SW_DPDT_x2, Eurorack:Sub-Miniature Toggle Switch DPDT, F.Cu at (10.0, 40.0)
- CONN1: footprint Eurorack:Header 2.0mm Right Angle Female -> Eurorack:Header 01x07 2.0mm Right Angle Female
- CONN2: footprint Eurorack:Header 2.0mm Right Angle Male -> Eurorack:Header 01x07 2.0mm Right Angle Male
- moved CONN1 67.4 mm to (0.00, 87.9)
- moved CONN2 65.4 mm to (20.0, 85.9)
- moved C1 13.5 mm to (2.53, 72.5)
- moved C2 13.5 mm to (17.5, 72.5)
- moved R1 7.37 mm to (2.03, 55.4)
- moved R2 7.37 mm to (18.0, 55.4)
- moved R3 7.37 mm to (2.03, 42.4)
- moved R4 7.37 mm to (18.0, 42.4)
- moved VR1 6.12 mm to (10.0, 78.9)
- moved P1 5.77 mm to (10.0, 32.0)
Connections:
- CONN1 pad 1: Net-(CONN1-Pad1) -> /LEFT BUS
- CONN1 pad 2: Net-(CONN1-Pad2) -> /RIGHT BUS
- CONN2 pad 1: /+12V -> Net-(CONN2-Pad1)
- CONN2 pad 2: Earth -> Net-(CONN2-Pad2)
- CONN2 pad 3: /-12V -> /+12V
- CONN2 pad 4: Net-(CONN1-Pad2) -> Earth
- CONN2 pad 5: Net-(CONN1-Pad1) -> /-12V
- R3 pad 2: Net-(CONN1-Pad1) -> /LEFT SIGNAL
- R4 pad 2: Net-(CONN1-Pad2) -> /RIGHT SIGNAL
Routing:
- net /LEFT BUS: track 0.00 -> 94.6 mm
- net /RIGHT BUS: track 0.00 -> 77.4 mm
- net Net-(CONN1-Pad2): track 18.7 -> 0.00 mm
- net Net-(CONN1-Pad1): track 17.6 -> 0.00 mm
- net Net-(J1-Pad3): track 69.9 -> 54.7 mm, vias 0 -> 2
- net Net-(CONN2-Pad2): track 0.00 -> 12.7 mm
- net Net-(CONN2-Pad1): track 0.00 -> 12.7 mm
- net Net-(P1-Pad3): track 15.7 -> 27.8 mm
- net Net-(P1-Pad1): track 18.7 -> 29.8 mm
- net /LEFT SIGNAL: track 0.00 -> 9.80 mm
- net /RIGHT SIGNAL: track 0.00 -> 8.94 mm
- net Net-(C2-Pad2): track 4.46 -> 10.6 mm
- net Net-(C1-Pad2): track 4.46 -> 10.6 mm
- net Net-(C1-Pad1): track 15.8 -> 21.1 mm
- net Net-(C2-Pad1): track 41.3 -> 36.3 mm
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Other:
- outline, holes or cut-outs redrawn
- board text added: "FX LEFT"
- board text added: "FX RIGHT"
- board text removed: "MALE"
- board text removed: "SCREW: M2.5x6mm"
- board text removed: "STANDOFF: M2.5x10mm"

Commit message: Changes
Parts:
- CONN1: footprint Eurorack:Header 01x07 2.0mm Right Angle Female -> Eurorack:Header 01x12 2.0mm Right Angle Female
- CONN2: footprint Eurorack:Header 01x07 2.0mm Right Angle Male -> Eurorack:Header 01x12 2.0mm Right Angle Male
- moved R2 21.6 mm to (1.52, 41.4)
- moved C2 14.8 mm to (2.79, 71.9)
- moved C1 14.8 mm to (17.3, 71.9)
- moved R1 14.1 mm to (4.06, 41.4)
- moved R3 14.0 mm to (16.0, 41.4), turned to -90 degrees
- moved CONN2 2.00 mm to (20.0, 87.9)
- moved R4 1.09 mm to (18.5, 41.4), turned to -90 degrees
- moved P1 0.61 mm to (10.0, 31.4)
Connections:
- CONN1 pad 6: Net-(CONN2-Pad2) -> Net-(CONN1-Pad6)
- CONN1 pad 7: Net-(CONN2-Pad1) -> Net-(CONN1-Pad7)
- CONN2 pad 1: Net-(CONN2-Pad1) -> Net-(CONN1-Pad12)
- CONN2 pad 2: Net-(CONN2-Pad2) -> Net-(CONN1-Pad11)
- CONN2 pad 3: /+12V -> Net-(CONN1-Pad10)
- CONN2 pad 4: Earth -> Net-(CONN1-Pad9)
- CONN2 pad 5: /-12V -> Net-(CONN1-Pad8)
- CONN2 pad 6: /RIGHT BUS -> Net-(CONN1-Pad7)
- CONN2 pad 7: /LEFT BUS -> Net-(CONN1-Pad6)
Routing:
- net Net-(P1-Pad1): track 29.8 -> 70.7 mm
- net Net-(C1-Pad2): track 10.6 -> 33.6 mm
- net /LEFT BUS: track 94.6 -> 72.8 mm
- net Earth: track 141.6 -> 157.8 mm
- net Net-(J1-Pad3): track 54.7 -> 70.5 mm, vias 2 -> 0
- net Net-(C2-Pad2): track 10.6 -> 24.2 mm
- net Net-(CONN1-Pad9): track 0.00 -> 12.8 mm
- net Net-(CONN2-Pad2): track 12.7 -> 0.00 mm
- net Net-(CONN2-Pad1): track 12.7 -> 0.00 mm
- net Net-(CONN1-Pad8): track 0.00 -> 12.7 mm
- net Net-(CONN1-Pad7): track 0.00 -> 12.7 mm
- net Net-(CONN1-Pad6): track 0.00 -> 12.7 mm
- net Net-(CONN1-Pad12): track 0.00 -> 12.7 mm
- net Net-(CONN1-Pad11): track 0.00 -> 12.7 mm
- net Net-(CONN1-Pad10): track 0.00 -> 12.7 mm
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Other:
- board text added: "stackable mixer www.allensynthesis.co.uk CERN OHL-S v2 Designed in Loughborough, UK 03/04/2022"
- board text removed: "1uF"
- board text removed: "FX LEFT"
- board text removed: "FX RIGHT"
