File: hardware/kicad-individual-channel/Stackable Mixer.kicad_sch (KiCad schematic)
At the start: 12 parts, among them J1 L/Mono, J2 R, P1 Potentiometer_9mm_Vertical_Li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

Commit message: Changes
Parts:
- added SW1: SW_DPDT_x2, Eurorack:Sub-Miniature Toggle Switch DPDT, symbol Switch:SW_DPDT_x2
- CONN1: footprint Eurorack:Header 2.0mm Right Angle Female -> Eurorack:Header 01x07 2.0mm Right Angle Female; symbol Eurorack:Header_2.0mm_Right_Angle_Female -> Eurorack:Header_01x07_2.0mm_Right_Angle_Female
- CONN2: footprint Eurorack:Header 2.0mm Right Angle Male -> Eurorack:Header 01x07 2.0mm Right Angle Male; symbol Eurorack:Header_2.0mm_Right_Angle_Male -> Eurorack:Header_01x07_2.0mm_Right_Angle_Female
Connections:
- net +12V: now also CONN2.3; no longer CONN2.1
- net -12V: now also CONN2.5; no longer CONN2.3
- net Earth: now also CONN2.4; no longer CONN2.2
- new net: CONN1.7, CONN2.1
- new net: CONN1.6, CONN2.2
- new net LEFT BUS: CONN1.1, CONN2.7, SW1.1 (A)
- new net LEFT SIGNAL: R3.2, SW1.2 (B)
- new net RIGHT BUS: CONN1.2, CONN2.6, SW1.4 (A)
- new net RIGHT SIGNAL: R4.2, SW1.5 (B)
- no-connect marks 0 -> 2

Commit message: Changes
Parts:
- CONN1: footprint Eurorack:Header 01x07 2.0mm Right Angle Female -> Eurorack:Header 01x12 2.0mm Right Angle Female; symbol Eurorack:Header_01x07_2.0mm_Right_Angle_Female -> Eurorack:Header_01x12_2.0mm_Right_Angle_Female
- CONN2: footprint Eurorack:Header 01x07 2.0mm Right Angle Male -> Eurorack:Header 01x12 2.0mm Right Angle Male; symbol Eurorack:Header_01x07_2.0mm_Right_Angle_Female -> Eurorack:Header_01x12_2.0mm_Right_Angle_Female
- P1: value Potentiometer_9mm_Vertical_Linear -> 100K
- R3, R4: value 4.7k -> 100k
Connections:
- net +12V: now also CONN2.8; no longer CONN2.3
- net -12V: now also CONN2.10; no longer CONN2.5
- net Earth: now also CONN2.9; no longer CONN2.4
- net LEFT BUS: now also CONN2.12; no longer CONN2.7
- net RIGHT BUS: now also CONN2.11; no longer CONN2.6
- net at CONN2.1: now also CONN1.12; no longer CONN1.7
- net at CONN2.2: now also CONN1.11; no longer CONN1.6
- new net: CONN1.10, CONN2.3
- new net: CONN1.9, CONN2.4
- new net: CONN1.8, CONN2.5
- new net: CONN1.7, CONN2.6
- new net: CONN1.6, CONN2.7
Changed lines of the file:
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@@
+    (stroke (width 0) (type default) (color 0 0 0 0))
+  )
+  (wire (pts (xy 162.56 151.13) (xy 181.61 151.13))
     (stroke (width 0) (type default) (color 0 0 0 0))
   )
@@
     (stroke (width 0) (type default) (color 0 0 0 0))
   )
+  (wire (pts (xy 162.56 140.97) (xy 181.61 140.97))
+    (stroke (width 0) (type default) (color 0 0 0 0))
+  )
   (wire (pts (xy 178.435 72.39) (xy 178.435 97.155))
     (stroke (width 0) (type default) (color 0 0 0 0))
@@
     (stroke (width 0) (type default) (color 0 0 0 0))
   )
+  (wire (pts (xy 162.56 143.51) (xy 181.61 143.51))
+    (stroke (width 0) (type default) (color 0 0 0 0))
+  )
   (wire (pts (xy 167.005 125.73) (xy 181.61 125.73))
     (stroke (width 0) (type default) (color 0 0 0 0))
@@
     (stroke (width 0) (type default) (color 0 0 0 0))
   )
+  (wire (pts (xy 162.56 146.05) (xy 181.61 146.05))
+    (stroke (width 0) (type default) (color 0 0 0 0))
+  )
   (wire (pts (xy 162.56 128.27) (xy 167.005 128.27))
     (stroke (width 0) (type default) (color 0 0 0 0))
@@
   )
   (wire (pts (xy 69.85 76.2) (xy 78.74 76.2))
+    (stroke (width 0) (type default) (color 0 0 0 0))
+  )
+  (wire (pts (xy 162.56 148.59) (xy 181.61 148.59))
     (stroke (width 0) (type default) (color 0 0 0 0))
   )
@@
     (effects (font (size 1.27 1.27)) (justify left bottom))
   )
-  (symbol (lib_id "Eurorack:Header_01x07_2.0mm_Right_Angle_Female") (at 181.61 142.24 0) (mirror x) (unit 1)
+  (symbol (lib_id "Eurorack:Header_01x12_2.0mm_Right_Angle_Female") (at 181.61 154.94 0) (mirror x) (unit 1)
     (in_bom yes) (on_board yes)
-    (property "Reference" "CONN2" (id 0) (at 192.405 117.475 0))
-    (property "Value" "Header_2.0mm_Right_Angle_Male" (id 1) (at 192.405 120.015 0))
-    (property "Footprint" "Eurorack:Header 01x07 2.0mm Right Angle Male" (id 2) (at 181.61 142.24 0)
-      (effects (font (size 1.27 1.27)) hide)
-    )
-    (property "Datasheet" "" (id 3) (at 181.61 142.24 0)
-      (effects (font (size 1.27 1.27)) hide)
-    )
-    (pin "1")
+    (property "Reference" "CONN2" (id 0) (at 192.405 130.175 0))
+    (property "Value" "Header_2.0mm_Right_Angle_Male" (id 1) (at 192.405 132.715 0))
+    (property "Footprint" "Eurorack:Header 01x12 2.0mm Right Angle Male" (id 2) (at 181.61 154.94 0)
+      (effects (font (size 1.27 1.27)) hide)
+    )
+    (property "Datasheet" "" (id 3) (at 181.61 154.94 0)
+      (effects (font (size 1.27 1.27)) hide)
+    )
+    (pin "1")
+    (pin "10")
+    (pin "11")
+    (pin "12")
     (pin "2")
     (pin "3")
@@
     (pin "6")
     (pin "7")
-  )
-  (symbol (lib_id "Eurorack:Header_01x07_2.0mm_Right_Angle_Female") (at 162.56 119.38 0) (mirror y) (unit 1)
+    (pin "8")
+    (pin "9")
+  )
+  (symbol (lib_id "Eurorack:Header_01x12_2.0mm_Right_Angle_Female") (at 162.56 119.38 0) (mirror y) (unit 1)
     (in_bom yes) (on_board yes)
     (property "Reference" "CONN1" (id 0) (at 147.32 118.11 0))
     (property "Value" "Header_2.0mm_Right_Angle_Female" (id 1) (at 147.32 120.65 0))
-    (property "Footprint" "Eurorack:Header 01x07 2.0mm Right Angle Female" (id 2) (at 162.56 119.38 0)
+    (property "Footprint" "Eurorack:Header 01x12 2.0mm Right Angle Female" (id 2) (at 162.56 119.38 0)
       (effects (font (size 1.27 1.27)) hide)
     )
@@
     )
     (pin "1")
+    (pin "10")
+    (pin "11")
+    (pin "12")
     (pin "2")
     (pin "3")
@@
     (pin "6")
     (pin "7")
+    (pin "8")
+    (pin "9")
   )
   (symbol (lib_id "Device:R") (at 113.03 72.39 90) (unit 1)
@@
       (effects (font (size 1.27 1.27)) (justify right))
     )
-    (property "Value" "Potentiometer_9mm_Vertical_Linear" (id 1) (at 127 68.58 90)
+    (property "Value" "100K" (id 1) (at 127 68.58 90)
       (effects (font (size 1.27 1.27)) (justify right))
     )
@@
     (in_bom yes) (on_board yes) (fields_autoplaced)
     (property "Reference" "R3" (id 0) (at 142.24 66.04 90))
-    (property "Value" "4.7k" (id 1) (at 142.24 68.58 90))
+    (property "Value" "100k" (id 1) (at 142.24 68.58 90))
     (property "Footprint" "Eurorack:Resistor 0.25W Through-Hole" (id 2) (at 142.24 74.168 90)
       (effects (font (size 1.27 1.27)) hide)
@@
     (in_bom yes) (on_board yes) (fields_autoplaced)
     (property "Reference" "R4" (id 0) (at 142.24 78.74 90))
-    (property "Value" "4.7k" (id 1) (at 142.24 81.28 90))
+    (property "Value" "100k" (id 1) (at 142.24 81.28 90))
     (property "Footprint" "Eurorack:Resistor 0.25W Through-Hole" (id 2) (at 142.24 86.868 90)
       (effects (font (size 1.27 1.27)) hide)
@@
     )
     (path "/38f9c384-4341-4365-9b6d-e2436e815ca3"
-      (reference "CONN1") (unit 1) (value "Header_2.0mm_Right_Angle_Female") (footprint "Eurorack:Header 01x07 2.0mm Right Angle Female")
+      (reference "CONN1") (unit 1) (value "Header_2.0mm_Right_Angle_Female") (footprint "Eurorack:Header 01x12 2.0mm Right Angle Female")
     )
     (path "/285a8d13-490e-40ca-ae74-b8e899d2c383"
-      (reference "CONN2") (unit 1) (value "Header_2.0mm_Right_Angle_Male") (footprint "Eurorack:Header 01x07 2.0mm Right Angle Male")
+      (reference "CONN2") (unit 1) (value "Header_2.0mm_Right_Angle_Male") (footprint "Eurorack:Header 01x12 2.0mm Right Angle Male")
     )
     (path "/69b87c2a-3f10-4e7b-944c-caf508f585eb"
@@
     )
     (path "/5d8c5941-87eb-4da1-9593-333289a9fd19"
-      (reference "P1") (unit 1) (value "Potentiometer_9mm_Vertical_Linear") (footprint "Eurorack:Potentiometer 9mm Vertical Linear")
+      (reference "P1") (unit 1) (value "100K") (footprint "Eurorack:Potentiometer 9mm Vertical Linear")
     )
     (path "/4545d90c-1e8d-4776-805c-dce54bf3d01b"
@@
     )
     (path "/92592b85-3719-4db8-9d54-3873879581aa"
-      (reference "R3") (unit 1) (value "4.7k") (footprint "Eurorack:Resistor 0.25W Through-Hole")
+      (reference "R3") (unit 1) (value "100k") (footprint "Eurorack:Resistor 0.25W Through-Hole")
     )
     (path "/b656d0b6-ba6e-4a59-9fb1-ff442dbfba37"
-      (reference "R4") (unit 1) (value "4.7k") (footprint "Eurorack:Resistor 0.25W Through-Hole")
+      (reference "R4") (unit 1) (value "100k") (footprint "Eurorack:Resistor 0.25W Through-Hole")
     )
     (path "/4b7f481a-ffab-49b6-ab70-058e45c84eb0"
