File: hardware/kicad-output-stage/Summing Stage.kicad_sch (KiCad schematic)
At the start: 18 parts, among them IC1 TL074, J1 Thonkiconn_Mono_Jack, J2 AudioJack3

Commit message: Changes
Parts:
- added C5, C6: 100n, Capacitor_THT:C_Disc_D4.7mm_W2.5mm_P5.00mm, symbol Device:C
- added SW1: SW_DPDT_x2, Eurorack:Sub-Miniature Toggle Switch DPDT, symbol Switch:SW_DPDT_x2
- CONN1: footprint Eurorack:Header 2.0mm Right Angle Female -> Eurorack:Header 01x12 2.0mm Right Angle Female; symbol Eurorack:Header_2.0mm_Right_Angle_Female -> Eurorack:Header_01x12_2.0mm_Right_Angle_Female
- R3, R4: value 4.7k -> 47K
- R5, R6: value 4.7k -> 100K
- VR1: value Potentiometer_45mm_Slide_Audio_Dual -> 100K
Connections:
- net L OUT: now also SW1.1 (A); no longer R1.2
- net R OUT: now also SW1.4 (A); no longer R2.2
- new net: C5.1, R1.2
- new net: C5.2, SW1.2 (B)
- new net: C6.2, SW1.5 (B)
- new net: C6.1, R2.2
- no-connect marks 2 -> 4
Other:
- moved on the sheet: D1, D2, J1, J2, PowerHeader1, R1, R2
